Commit message: second committt

File: Isaaclab_other/agent_for_isaaclab/urdf/current_agent.urdf (robot description, URDF)
Before this commit: robot initial_agent_hand, 21 links, 20 joints
Links:
- removed link link_3_3_child_deb4d61f
- removed link link_4_3_child_e4e32045
- removed link link_5_3_child_67d97dfa
- added link link_2_2, mass 0.1; collision mesh filename=/home/qyx/Desktop/Isaaclab_other/agent_for_isaaclab/mesh/li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; visual mesh filename=/home/qyx/Desktop/Isaaclab_other/agent_for_isaaclab/mesh/li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
- added link link_2_3, mass 0.1; collision mesh filename=/home/qyx/Desktop/Isaaclab_other/agent_for_isaaclab/mesh/li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; visual mesh filename=/home/qyx/Desktop/Isaaclab_other/agent_for_isaaclab/mesh/li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
Joints:
- removed joint link_3_3_to_link_3_3_child_deb4d61f
- removed joint link_4_3_to_link_4_3_child_e4e32045
- removed joint link_5_3_to_link_5_3_child_67d97dfa
- added joint link_2_1_to_link_2_2: type revolute, parent link_2_1, child link_2_2, origin xyz=0.0 0.0 0.032 rpy=0.0 -0.0 0.0, axis 1. 0. 0., limit lower=0.0 upper=1.57 effort=5.0 velocity=1.5
- added joint link_2_2_to_link_2_3: type revolute, parent link_2_2, child link_2_3, origin xyz=0.0 0.0 0.024 rpy=0.0 -0.0 0.0, axis 1. 0. 0., limit lower=0.0 upper=1.57 effort=5.0 velocity=1.5

File: Isaaclab_other/agent_for_isaaclab_mirror/urdf/current_agent.urdf (robot description, URDF)
Before this commit: robot mirror_agent_hand, 21 links, 20 joints
Links:
- removed link link_3_3_child_deb4d61f
- removed link link_4_3_child_e4e32045
- removed link link_5_3_child_67d97dfa
- added link link_2_2, mass 0.1; collision mesh filename=/home/qyx/Desktop/Isaaclab_other/agent_for_isaaclab_mirror/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; visual mesh filename=/home/qyx/Desktop/Isaaclab_other/agent_for_isaaclab_mirror/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
- added link link_2_3, mass 0.1; collision mesh filename=/home/qyx/Desktop/Isaaclab_other/agent_for_isaaclab_mirror/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; visual mesh filename=/home/qyx/Desktop/Isaaclab_other/agent_for_isaaclab_mirror/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
Joints:
- removed joint link_3_3_to_link_3_3_child_deb4d61f
- removed joint link_4_3_to_link_4_3_child_e4e32045
- removed joint link_5_3_to_link_5_3_child_67d97dfa
- added joint link_2_1_to_link_2_2: type revolute, parent link_2_1, child link_2_2, origin xyz=0.0 0.0 0.032 rpy=0.0 -0.0 0.0, axis 1. 0. 0., limit lower=0.0 upper=1.57 effort=5.0 velocity=1.5
- added joint link_2_2_to_link_2_3: type revolute, parent link_2_2, child link_2_3, origin xyz=0.0 0.0 0.024 rpy=0.0 -0.0 0.0, axis 1. 0. 0., limit lower=0.0 upper=1.57 effort=5.0 velocity=1.5
